File: KiCad_Traffic_Light_Controller_guide/KiCad_JLPCB_template_2layers/Traffic_Light_Controller/Traffic_Light_Controller.kicad_pcb (KiCad board)
At the start: 2 copper layers, 124.2 x 91.4 mm, 65 parts, among them J1 Conn_02x08_Odd_Even, J2 Conn_02x08_Odd_Even, J3 Conn_02x05_Odd_Even, J4 +5V, SW1 RST, SW2 OVRRIDE, SW3 EN, U1 SM420561N, U2 SM420561N, U3 LM1117DT-3.3

Commit message: n
Parts:
- removed the G*** at (182.8, 135.6)
- added G***: LOGO, LOGO, F.Cu at (188.0, 135.5)
- added G***: LOGO, LOGO, F.Cu at (148.0, 136.5)
Other:
- board text added: "Jaena, Elaiza B. 19 April 2026 Computer Engineering Technology Department Technological University of the Philippines-Visayas"
- board text removed: "Cid Lawrenc C. Regalado 19 April 2026 Computer Engineering Technology Department Technological University of the Philippines-Visayas"

Commit message: commit
Parts:
- removed the G*** at (188.0, 135.5)
- removed the G*** at (148.0, 136.5)
- added G***: LOGO, LOGO, F.Cu at (161.5, 135.0)
- added G***: LOGO, LOGO, F.Cu at (204.5, 134.0)
- moved C4 15.0 mm to (114.0, 80.0)
- moved D10 15.0 mm to (102.2, 127.3)
- moved D11 15.0 mm to (186.4, 114.9)
- moved D13 15.0 mm to (169.5, 114.6)
- moved D2 15.0 mm to (168.6, 73.1)
- moved D4 15.0 mm to (132.1, 109.1)
- moved D5 15.0 mm to (132.1, 119.7)
- moved D6 15.0 mm to (132.1, 130.2)
- moved D7 15.0 mm to (201.0, 67.7)
- moved H2 15.0 mm to (211.3, 55.3)
- moved H4 15.0 mm to (93.3, 140.4)
- moved J1 15.0 mm to (125.9, 75.8)
- moved J3 15.0 mm to (133.4, 63.3)
- moved J4 15.0 mm to (103.8, 63.6)
- moved R1 15.0 mm to (186.8, 59.8)
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Routing:
- net /+3.3V: track 281.7 -> 279.3 mm
- net /OVR: track 131.4 -> 129.7 mm
- net /NS_HEX_A: track 106.3 -> 107.8 mm
- net GND: track 467.1 -> 465.6 mm
- net /EN: track 146.5 -> 147.8 mm
Other:
- board size 124.2 x 91.4 mm -> 124.2 x 91.3 mm
- board text added: "Jaena, Elaiza B. 19 April 2026 Computer Engineering Technology Department Technological University of the Philippines Visayas"
- board text removed: "Jaena, Elaiza B. 19 April 2026 Computer Engineering Technology Department Technological University of the Philippines-Visayas"
